Commit message: updated version of Go1_description

File: go1_simulation/go1_description/xacro/robot.xacro (robot description, xacro)
@@ -10,4 +10,6 @@
     <xacro:include filename="$(find go1_description)/xacro/Accessories/rplidar.xacro"/>
     <xacro:property name="M_PI" value="3.1415926535897931" />
+    <xacro:arg name="with_lidar" default="true" />
+    <xacro:arg name="DEBUG" default="false" />
     <!-- Rollover Protection mode will add an additional stick on the top, use "true" or "false" to switch it. -->
     <xacro:property name="rolloverProtection" value="false"/>
@@ -161,6 +163,8 @@
         <origin rpy="0 0 0" xyz="0.2747 0.0 -0.0088"/>
     </xacro:ultraSound>
-    <xacro:rplidar>
-        <origin xyz="0.140468617087559 0 0.057" rpy="0 0 0.000119868886667814"/>
-    </xacro:rplidar>
+    <xacro:if value="$(arg with_lidar)">
+        <xacro:rplidar>
+            <origin xyz="0.140468617087559 0 0.057" rpy="0 0 0.000119868886667814"/>
+        </xacro:rplidar>
+    </xacro:if>
 </robot>

File: unitree_go1_hw_ros/go1_description/xacro/gazebo.xacro (robot description, xacro)
@@ -126,5 +126,5 @@
         </sensor>
     </gazebo> -->
-  <gazebo reference="depthCamera_link_left">
+<!--   <gazebo reference="depthCamera_link_left">
     <sensor name="camera_link_camera" type="depth">
       <update_rate>20</update_rate>
@@ -167,4 +167,5 @@
     </sensor>
   </gazebo>
+ -->
     <!-- Foot contacts. -->
     <gazebo reference="FR_calf">
